File: posey-hx.kicad_sch (KiCad schematic)
At the start: 31 parts, among them J1 TC2050-IDC-NL, U1 NORA-B106-00B, U2 W25N01GVZEIG_TR, Y1 XTAL, Y2 XTAL

Commit message: Updated readme, license, and version.
Parts:
- added C11: 0.1µ, Capacitor_SMD:C_0402_1005Metric, symbol Device:C
- added J2: Conn_02x06_Odd_Even, Connector_PinHeader_1.27mm:PinHeader_2x06_P1.27mm_Vertical, symbol Connector_Generic:Conn_02x06_Odd_Even
- IMU1: value BNO080 -> BNO085/6
- J1, LiPo1, Vin1: now left out of the parts list
- R10, R12: now not fitted; now left out of the parts list
Connections:
- net GND: now also C11.2, J2.7 (Pin_7), J2.9 (Pin_9); no longer IMU1.5 (PS1), IMU1.6 (PS0/WAKE)
- net IMU_nINT: now also J2.3 (Pin_3)
- net IMU_nRESET: now also J2.2 (Pin_2)
- net SCL/SPI_SCK: now also J2.12 (Pin_12)
- net SDA/SPI_CIPO: now also J2.10 (Pin_10)
- net SPI_COPI: now also J2.6 (Pin_6)
- net SPI_CS_IMU: now also J2.8 (Pin_8)
- net VBAT: now also J2.11 (Pin_11)
- net VCC: now also C11.1, J2.1 (Pin_1)
- net IMU_PS1: now reaches U1.A5 (P0.20)
- net IMU_PS1: now also IMU1.5 (PS1), J2.4 (Pin_4)
- net IMU_PS0: now reaches U1.C4 (P1.01)
- net IMU_PS0: now also IMU1.6 (PS0/WAKE), J2.5 (Pin_5)
Other:
- note removed: "2023.10.18"
- note removed: "2310"
- note removed: "Posey IMU Platform"
- note removed: "Soft Machines Lab Carnegie Mellon University License here"
- company: (none) -> Soft Machines Lab
- title: (none) -> Posey Hub
